File: DistributionBoard/eagle/DistributionBoard.sch (EAGLE design)
At the start: 53 parts, among them X1 22-23-2031, X10 22-23-2041, X11 22-23-2031, X12 22-23-2031, X13 22-23-2031, X14 22-23-2031, X15 22-23-2031, X16 22-23-2031, X17 22-23-2031, X18 22-23-2031, X19 22-23-2031, X2 22-23-2031, X20 22-23-2031, X3 22-23-2031, X4 22-23-2031, X5 22-23-2031, X6 22-23-2031, X7 22-23-2041, X8 22-23-2041, X9 22-23-2041

Commit message: Distribution Board
Parts:
- added Q1, Q2, Q3, Q4: BC639, transistor-small-signal:BC639
- added R1, R2, R3, R4: 330, rcl:R-EU_M1206
- added R5: 10k, rcl:R-EU_M1206
- added R6, R7, R8: 10K, rcl:R-EU_M1206
Connections:
- new net N$10: Q3.B, R3.2
- new net N$11: Q2.B, R2.2
- new net N$12: Q1.B, R1.2
- new net N$9: Q4.B, R4.2
- new net S1: Q1.C, X17-1.S
- new net S2: Q2.C, X18-1.S
- new net S3: Q3.C, X19-1.S
- new net S4: Q4.C, X20-1.S
- net D28: now also R1.1, R5.1
- net D29: now also R2.1, R6.1
- net D30: now also R3.1, R7.1
- net D31: now also R4.1, R8.1
- net GND: now also Q1.E, Q2.E, Q3.E, Q4.E, R5.2, R6.2, R7.2, R8.2; no longer X17-1.S, X18-1.S, X19-1.S, X20-1.S
Other:
- moved on the sheet: +5V, 7850, C1, LED1, LED2, LED3, LED4, LED5, LED6, RESET, RN1, T1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
