File: DistributionBoard/eagle/DistributionBoard.brd (EAGLE design)
At the start: 120 x 64.8 mm, 53 parts, among them X1 22-23-2031, X10 22-23-2041, X11 22-23-2031, X12 22-23-2031, X13 22-23-2031, X14 22-23-2031, X15 22-23-2031, X16 22-23-2031, X17 22-23-2031, X18 22-23-2031, X19 22-23-2031, X2 22-23-2031, X20 22-23-2031, X3 22-23-2031, X4 22-23-2031, X5 22-23-2031, X6 22-23-2031, X7 22-23-2041, X8 22-23-2041, X9 22-23-2041

Commit message: Distribution Board
Parts:
- added Q1, Q2, Q3, Q4: BC639, transistor-small-signal:SOT54D
- added R1, R2, R3, R4: 330, rcl:M1206
- added R5: 10k, rcl:M1206
- added R6, R7, R8: 10K, rcl:M1206
Connections:
- new net N$10: Q3.B, R3.2
- new net N$11: Q2.B, R2.2
- new net N$12: Q1.B, R1.2
- new net N$9: Q4.B, R4.2
- new net S1: Q1.C, X17.1
- new net S2: Q2.C, X18.1
- new net S3: Q3.C, X19.1
- new net S4: Q4.C, X20.1
- net D28: now also R1.1, R5.1
- net D29: now also R2.1, R6.1
- net D30: now also R3.1, R7.1
- net D31: now also R4.1, R8.1
- net GND: now also Q1.E, Q2.E, Q3.E, Q4.E, R5.2, R6.2, R7.2, R8.2; no longer X17.1, X18.1, X19.1, X20.1
Routing:
- net D28: track 8.67 -> 97.9 mm
- net D29: track 8.67 -> 93.1 mm, vias 0 -> 1
- net D30: track 8.67 -> 81.5 mm
- net D31: track 8.67 -> 58.1 mm, vias 0 -> 1
- net VCC: track 26.1 -> 73.9 mm
- net +5V: track 391.1 -> 349.0 mm, vias 0 -> 3
- net D32: track 121.5 -> 128.0 mm
- net D33: track 120.8 -> 126.7 mm
- net D34: track 113.9 -> 119.3 mm
- net N$9: track 0.00 -> 5.21 mm
- net D35: track 113.2 -> 118.0 mm
- net S4: track 0.00 -> 4.45 mm
- net S3: track 0.00 -> 4.45 mm
- net S2: track 0.00 -> 4.45 mm
- net S1: track 0.00 -> 4.45 mm
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- added copper zone on layer 1, net GND
- added copper zone on layer 16, net GND
Other:
- board size 120 x 64.8 mm -> 119.4 x 64.8 mm
- board text added: "------------------------------- Input: 7V - 36V Output: 5V @ 2A I/O: 5V ONLY! ------------------------------- No Pullups on Buttons -------------------------------"
- board text added: "Distribution Board"
- board text added: "VCC"
- board text added: "Version 1.0.0"
- board text added: "drill ->"
- board text removed: "Distribution Board v.1"

Commit message: Distribution Board fertig
Routing:
- net +5V: vias 3 -> 4
Changed lines of the file:
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@@
 <attribute name="MF" value="" x="6.35" y="19.3675" size="1.778" layer="27" display="off"/>
 <attribute name="MPN" value="B3F-1000" x="6.35" y="19.3675" size="1.778" layer="27" display="off"/>
-<attribute name="NAME" x="10.287" y="18.6055" size="1.27" layer="25" ratio="10"/>
+<attribute name="NAME" x="0.762" y="18.6055" size="1.27" layer="25" ratio="10"/>
 <attribute name="OC_FARNELL" value="176432" x="6.35" y="19.3675" size="1.778" layer="27" display="off"/>
 <attribute name="OC_NEWARK" value="36M3542" x="6.35" y="19.3675" size="1.778" layer="27" display="off"/>
@@
 <attribute name="MF" value="" x="6.35" y="26.3525" size="1.778" layer="27" display="off"/>
 <attribute name="MPN" value="B3F-1000" x="6.35" y="26.3525" size="1.778" layer="27" display="off"/>
-<attribute name="NAME" x="10.287" y="25.5905" size="1.27" layer="25" ratio="10"/>
+<attribute name="NAME" x="0.762" y="25.5905" size="1.27" layer="25" ratio="10"/>
 <attribute name="OC_FARNELL" value="176432" x="6.35" y="26.3525" size="1.778" layer="27" display="off"/>
 <attribute name="OC_NEWARK" value="36M3542" x="6.35" y="26.3525" size="1.778" layer="27" display="off"/>
@@
 <attribute name="MF" value="" x="6.35" y="5.3975" size="1.778" layer="27" display="off"/>
 <attribute name="MPN" value="B3F-1000" x="6.35" y="5.3975" size="1.778" layer="27" display="off"/>
-<attribute name="NAME" x="10.287" y="4.6355" size="1.27" layer="25" ratio="10"/>
+<attribute name="NAME" x="0.762" y="4.6355" size="1.27" layer="25" ratio="10"/>
 <attribute name="OC_FARNELL" value="176432" x="6.35" y="5.3975" size="1.778" layer="27" display="off"/>
 <attribute name="OC_NEWARK" value="36M3542" x="6.35" y="5.3975" size="1.778" layer="27" display="off"/>
@@
 <attribute name="MF" value="" x="6.35" y="12.3825" size="1.778" layer="27" display="off"/>
 <attribute name="MPN" value="B3F-1000" x="6.35" y="12.3825" size="1.778" layer="27" display="off"/>
-<attribute name="NAME" x="10.287" y="11.6205" size="1.27" layer="25" ratio="10"/>
+<attribute name="NAME" x="0.762" y="11.6205" size="1.27" layer="25" ratio="10"/>
 <attribute name="OC_FARNELL" value="176432" x="6.35" y="12.3825" size="1.778" layer="27" display="off"/>
 <attribute name="OC_NEWARK" value="36M3542" x="6.35" y="12.3825" size="1.778" layer="27" display="off"/>
@@
 <via x="52.705" y="39.37" extent="1-16" drill="0.45"/>
 <via x="52.705" y="38.1" extent="1-16" drill="0.45"/>
-<wire x1="52.705" y1="38.1" x2="52.705" y2="39.37" width="2.032" layer="16"/>
 <wire x1="52.705" y1="39.37" x2="52.705" y2="40.3134" width="2.032" layer="16"/>
-<wire x1="52.705" y1="40.64" x2="52.705" y2="48.895" width="2.032" layer="16"/>
+<wire x1="52.705" y1="40.64" x2="52.705" y2="41.91" width="2.032" layer="16"/>
+<wire x1="52.705" y1="41.91" x2="52.705" y2="48.895" width="2.032" layer="16"/>
 <wire x1="52.705" y1="48.895" x2="56.515" y2="48.895" width="2.032" layer="16"/>
 <wire x1="56.515" y1="48.895" x2="63.5" y2="48.895" width="2.032" layer="16"/>
@@
 <wire x1="66.04" y1="51.435" x2="70.485" y2="51.435" width="2.032" layer="16"/>
 <wire x1="70.485" y1="51.435" x2="78.105" y2="51.435" width="2.032" layer="16"/>
-<wire x1="52.705" y1="40.64" x2="52.705" y2="39.37" width="2.032" layer="16"/>
+<wire x1="52.705" y1="39.37" x2="52.705" y2="40.64" width="1.524" layer="1"/>
+<via x="52.705" y="41.91" extent="1-16" drill="0.35"/>
+<wire x1="52.705" y1="39.37" x2="52.705" y2="38.1" width="1.143" layer="16"/>
 </signal>
 <signal name="+3.3V">
